File: pcb/WetCorn/WetCorn.kicad_pcb (KiCad board)
At the start: 2 copper layers, 118 x 90.6 mm, 100 parts, among them J1 USB_C Main, J2 USB_C I2C_L, J3 USB_C I2C_R, SW1 SW_Push, SW10 SW_Push, SW11 SW_Push, SW12 SW_Push, SW13 SW_Push, SW14 SW_Push, SW15 SW_Push, SW16 SW_Push, SW17 SW_Push, SW18 SW_Push, SW19 SW_Push, SW2 SW_Push, SW20 SW_Push, SW21 SW_Push, SW22 SW_Push, SW23 SW_Push, SW24 SW_Push, SW25 SW_Push, SW26 SW_Push, SW27 SW_Push, SW28 SW_Push, SW29 SW_Push, SW3 SW_Push, SW30 SW_Push, SW31 SW_Push, SW32 SW_Push, SW33 SW_Push, SW34 SW_Push, SW35 SW_Push, SW36 SW_Push, SW37 SW_Push, SW4 SW_Push, SW5 SW_Push, SW6 SW_Push, SW7 SW_Push, SW8 SW_Push, SW9 SW_Push, U1 SRV05-4, U2 TCA9555RTWR, U3 ATmega32U4-MU, Y1 16MHZ

Commit message: pcb wip
Parts:
- removed U1: SRV05-4, Package_TO_SOT_SMD:SOT-23-6
- J1, J2, J3: footprint WetCorn:USB_C 16 Pin -> WetCorn:USB-C-12-Pin-MidMount
- SW17, SW21, SW25, SW29: footprint WetCorn:Kailh_Choc_1.5u -> WetCorn:Kailh_Choc_1u
- moved D2 288.8 mm to (276.5, 42.6)
- moved SW17 273.7 mm to (225.8, 94.2), turned to 177 degrees
- moved U2 266.6 mm to (231.8, 83.3)
- moved SW25 265.2 mm to (204.9, 96.3), turned to 195 degrees
- moved SW33 258.5 mm to (182.3, 101.0), turned to 126 degrees
- moved SW29 252.2 mm to (122.9, 96.4), turned to 165 degrees
- moved SW37 250.8 mm to (145.5, 101.1), turned to 234 degrees
- moved D4 247.3 mm to (276.5, 76.6)
- moved SW16 238.6 mm to (240.5, 69.3)
- moved SW4 234.2 mm to (276.5, 81.3)
- moved SW32 232.7 mm to (204.5, 74.8)
- moved SW21 230.3 mm to (102.0, 94.2), turned to 183 degrees
- moved SW31 230.3 mm to (204.5, 57.8)
- moved SW3 229.2 mm to (276.5, 64.3)
- moved SW24 228.7 mm to (222.5, 72.3)
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Connections:
- R6 pad 1: Net-(R6-Pad1) -> /D-
- R6 pad 2: Net-(J1-PadA6) -> Net-(J1-PadA7)
- R7 pad 1: Net-(R7-Pad1) -> /D+
- R7 pad 2: Net-(J1-PadA7) -> Net-(J1-PadA6)
- U3 pad 3: Net-(R7-Pad1) -> /D-
- U3 pad 4: Net-(R6-Pad1) -> /D+
Routing:
- net /Row_R1: track 0.00 -> 88.2 mm
- net /Row_R2: track 0.00 -> 88.2 mm
- net /Row_R0: track 0.00 -> 88.2 mm
- net /Col_L3: track 0.00 -> 75.1 mm
- net /Col_L4: track 0.00 -> 71.0 mm
- net /Row_L0: track 0.00 -> 67.3 mm
- net /Row_L1: track 0.00 -> 63.6 mm
- net /Row_L2: track 0.00 -> 63.6 mm
- net /Row_R3: track 0.00 -> 53.6 mm
- net /Row_L3: track 0.00 -> 51.7 mm
- net /Col_L2: track 0.00 -> 50.1 mm
- net /Col_R0: track 0.00 -> 37.1 mm
- net /Col_R3: track 0.00 -> 37.1 mm
- net /Col_R4: track 0.00 -> 37.1 mm
- net /Col_R2: track 0.00 -> 37.1 mm
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Other:
- board size 118 x 90.6 mm -> 243.2 x 90.6 mm
- net class PWR added: clearance 0.2, trace_width 0.4, via_dia 0.8, via_drill 0.4

Commit message: PCB finished
Parts:
- added REF**: Breakaway_Tabs, kbd:Breakaway_Tabs, F.Cu at (276.6, 90.5)
- added REF**: Breakaway_Tabs, kbd:Breakaway_Tabs, F.Cu at (253.4, 90.5)
- added REF**: Breakaway_Tabs, kbd:Breakaway_Tabs, F.Cu at (73.6, 90.5)
- added REF**: Breakaway_Tabs, kbd:Breakaway_Tabs, F.Cu at (51.2, 90.5)
- added REF**: Breakaway_Tabs, kbd:Breakaway_Tabs, F.Cu at (258.5, 29.2)
- added REF**: Breakaway_Tabs, kbd:Breakaway_Tabs, F.Cu at (222.8, 29.2)
- added REF**: Breakaway_Tabs, kbd:Breakaway_Tabs, F.Cu at (105.2, 29.2)
- added REF**: Breakaway_Tabs, kbd:Breakaway_Tabs, F.Cu at (69.9, 29.2)
- C1, C2, C3, C4, C5, C6, C7, C8, C9: footprint Capacitor_SMD:C_0603_1608Metric_Pad1.08x0.95mm_HandSolder -> WetCorn:C_0402_HandSolder
- D1, D10, D11, D12, D13, D14, D15, D16, D17, D18, D19, D2, D20, D21, D22, D23, D24, D25, D26, D27, D28, D29, D3, D30, D31, D32, D33, D34, D35, D36, D37, D4, D5, D6, D7, D8, D9: footprint Diode_SMD:D_SOD-323_HandSoldering -> WetCorn:D_SOD-323_HandSoldering
- R1, R2, R3, R4, R5, R6, R7, R8, R9: footprint Resistor_SMD:R_0603_1608Metric_Pad0.98x0.95mm_HandSolder -> WetCorn:R_0402_HandSolder
- SW1: footprint Button_Switch_THT:SW_Tactile_SPST_Angled_PTS645Vx31-2LFS -> WetCorn:Micro_Push_Button_3x6x2.5mm
- moved C1 52.3 mm to (92.9, 85.6), turned to 315 degrees
- moved C2 48.8 mm to (92.8, 88.9), turned to 45 degrees
- moved Y1 42.9 mm to (91.1, 87.4), turned to 225 degrees
- moved R9 35.6 mm to (85.5, 77.4), turned to 180 degrees
- moved C7 32.6 mm to (88.7, 82.2), turned to 135 degrees
- moved C8 26.8 mm to (78.1, 75.8), turned to 45 degrees
- moved C6 23.7 mm to (78.8, 76.5), turned to 45 degrees
- moved C4 20.4 mm to (76.6, 81.5), turned to 315 degrees
- moved U3 17.0 mm to (82.8, 82.9), turned to 45 degrees
- moved R8 16.5 mm to (87.5, 87.8), turned to 315 degrees
- moved R5 15.0 mm to (228.4, 84.0), turned to 270 degrees
- moved C3 14.1 mm to (226.7, 83.4)
- moved C5 11.4 mm to (76.7, 87.0)
- moved D1 11.2 mm to (86.5, 88.9), turned to 315 degrees
- moved C9 4.16 mm to (76.7, 86.0)
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Connections:
- U2 pad 1: /Col_R0 -> /Col_R4
- U2 pad 13: /Row_R3 -> /Col_R1
- U2 pad 14: Net-(U2-Pad14) -> /Col_R2
- U2 pad 2: /Col_R1 -> /Col_R3
- U2 pad 3: /Col_R2 -> Net-(U2-Pad3)
- U2 pad 4: /Col_R3 -> Net-(U2-Pad4)
- U2 pad 5: /Col_R4 -> Net-(U2-Pad5)
- U2 pad 6: Net-(U2-Pad6) -> /Row_R3
- U2 pad 7: Net-(U2-Pad7) -> /Col_R0
- U3 pad 1: Net-(U3-Pad1) -> /Col_L1
- U3 pad 11: /Row_L3 -> /Col_L0
- U3 pad 12: /Col_L3 -> Net-(U3-Pad12)
- U3 pad 28: /Col_L0 -> /Row_L3
- U3 pad 29: /Col_L1 -> /Col_L4
- U3 pad 30: /Col_L2 -> /Col_L3
- U3 pad 31: /Col_L4 -> Net-(U3-Pad31)
- U3 pad 36: Net-(U3-Pad36) -> /Col_L2
Routing:
- net +5V: track 0.00 -> 175.0 mm, vias 0 -> 10
- net /Row_L0: track 67.3 -> 154.6 mm, vias 0 -> 2
- net /Row_L1: track 63.6 -> 137.8 mm, vias 0 -> 2
- net /Row_R0: track 88.2 -> 161.8 mm, vias 0 -> 2
- net /Col_R4: track 37.1 -> 99.5 mm, vias 0 -> 1
- net /I2C_SCL_L: track 0.00 -> 62.2 mm, vias 0 -> 2
- net /I2C_SDA_L: track 0.00 -> 60.7 mm, vias 0 -> 2
- net VDD: track 0.00 -> 57.7 mm, vias 0 -> 3
- net /Row_L2: track 63.6 -> 119.2 mm, vias 0 -> 2
- net /Row_R1: track 88.2 -> 143.8 mm, vias 0 -> 2
- net /I2C_SDA_R: track 0.00 -> 49.0 mm, vias 0 -> 2
- net /I2C_SCL_R: track 0.00 -> 48.0 mm, vias 0 -> 2
- net GND: track 2.63 -> 45.2 mm, vias 2 -> 18
- net /Col_R3: track 37.1 -> 79.7 mm, vias 0 -> 1
- net /Col_L0: track 37.1 -> 76.5 mm
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- added copper zone on B.Cu, net GND
- added copper zone on B.Cu, net VSS
Other:
- board size 243.2 x 90.6 mm -> 243.2 x 106 mm
- net class Default: clearance 0.2 -> 0.199
- net class PWR: clearance 0.2 -> 0.199
- rule trace_clearance: 0.2 -> 0.199
