File: pcb/3W6.kicad_pcb (KiCad board)
At the start: 2 copper layers, 243.2 x 106 mm, 107 parts, among them J1 USB_C Main, J2 USB_C I2C_L, J3 USB_C I2C_R, SW1 SW_Push, SW10 SW_Push, SW11 SW_Push, SW12 SW_Push, SW13 SW_Push, SW14 SW_Push, SW15 SW_Push, SW16 SW_Push, SW17 SW_Push, SW18 SW_Push, SW19 SW_Push, SW2 SW_Push, SW20 SW_Push, SW21 SW_Push, SW22 SW_Push, SW23 SW_Push, SW24 SW_Push, SW25 SW_Push, SW26 SW_Push, SW27 SW_Push, SW28 SW_Push, SW29 SW_Push, SW3 SW_Push, SW30 SW_Push, SW31 SW_Push, SW32 SW_Push, SW33 SW_Push, SW34 SW_Push, SW35 SW_Push, SW36 SW_Push, SW37 SW_Push, SW4 SW_Push, SW5 SW_Push, SW6 SW_Push, SW7 SW_Push, SW8 SW_Push, SW9 SW_Push, U2 TCA9555RTWR, U3 ATmega32U4-MU, Y1 16MHZ

Commit message: fixing some outlines
Parts:
- removed the REF** at (276.6, 90.5)
- removed the REF** at (253.4, 90.5)
- removed the REF** at (73.6, 90.5)
- removed the REF** at (51.2, 90.5)
- removed the REF** at (258.5, 29.2)
- removed the REF** at (222.8, 29.2)
- removed the REF** at (105.2, 29.2)
- removed the REF** at (69.9, 29.2)
- added D38: D, WetCorn:D_SOD-123, F.Cu at (46.2, 55.9)
- added D39: D, WetCorn:D_SOD-123, F.Cu at (46.2, 72.8)
- added D40: D, WetCorn:D_SOD-123, F.Cu at (128.5, 49.4)
- added D41: D, WetCorn:D_SOD-123, F.Cu at (78.2, 33.4)
- added D42: D, WetCorn:D_SOD-123, F.Cu at (128.5, 66.3)
- added D43: D, WetCorn:D_SOD-123, F.Cu at (199.5, 49.4)
- added D44: D, WetCorn:D_SOD-123, F.Cu at (96.2, 35.4)
- added D45: D, WetCorn:D_SOD-123, F.Cu at (87.0, 60.9)
- added D46: D, WetCorn:D_SOD-123, F.Cu at (249.5, 35.4)
- added D47: D, WetCorn:D_SOD-123, F.Cu at (199.5, 66.3)
- added D48: D, WetCorn:D_SOD-123, F.Cu at (134.2, 97.8)
- added D49: D, WetCorn:D_SOD-123, F.Cu at (193.0, 96.8)
- added D50: D, WetCorn:D_SOD-123, F.Cu at (231.5, 33.4)
- added D51: D, WetCorn:D_SOD-123, F.Cu at (281.5, 72.8)
- added D52: D, WetCorn:D_SOD-123, F.Cu at (240.5, 60.9)
- added D53: D, WetCorn:D_SOD-123, F.Cu at (281.5, 55.9)
- added REF**: Breakaway_Tabs, kbd:Breakaway_Tabs, F.Cu at (276.6, 90.5)
- added REF**: Breakaway_Tabs, kbd:Breakaway_Tabs, F.Cu at (253.4, 90.5)
- added REF**: Breakaway_Tabs, kbd:Breakaway_Tabs, F.Cu at (73.7, 90.5)
- added REF**: Breakaway_Tabs, kbd:Breakaway_Tabs, F.Cu at (51.2, 90.5)
- added REF**: Breakaway_Tabs, kbd:Breakaway_Tabs, F.Cu at (258.5, 29.2)
- added REF**: Breakaway_Tabs, kbd:Breakaway_Tabs, F.Cu at (222.8, 29.2)
- added REF**: Breakaway_Tabs, kbd:Breakaway_Tabs, F.Cu at (105.2, 29.2)
- added REF**: Breakaway_Tabs, kbd:Breakaway_Tabs, F.Cu at (69.9, 29.2)
- C3: value 0.1u -> 0.1uF
- D1, D10, D11, D12, D13, D14, D15, D16, D17, D18, D19, D2, D20, D21, D22, D23, D24, D25, D26, D27, D28, D29, D3, D30, D31, D32, D33, D34, D35, D36, D37, D4, D5, D6, D7, D8, D9: footprint WetCorn:D_SOD-323_HandSoldering -> WetCorn:D_SOD-123
- F1: footprint Fuse:Fuse_1206_3216Metric_Pad1.42x1.75mm_HandSolder -> Fuse:Fuse_1206_3216Metric
- Y1: footprint Oscillator:Oscillator_SMD_Abracon_ASE-4Pin_3.2x2.5mm -> Crystal:Crystal_SMD_3225-4Pin_3.2x2.5mm
- moved C1 0.82 mm to (93.0, 84.8)
- moved C2 0.70 mm to (92.8, 88.2)
- moved Y1 0.70 mm to (91.1, 86.7)
- moved R8 0.56 mm to (88.0, 88.1)
- moved D1 0.39 mm to (86.7, 89.2)
Routing:
- net Net-(U3-Pad20): track 3.43 -> 0.00 mm, vias 1 -> 0
- net GND: track 45.2 -> 46.5 mm, vias 18 -> 17
- net +5V: track 175.0 -> 176.1 mm
- net /Row_L3: track 87.7 -> 86.6 mm
- net /Row_L1: track 137.8 -> 136.9 mm
- net /Row_R2: track 124.6 -> 124.0 mm
- net /Row_R3: track 71.9 -> 71.4 mm
