File: pcb/3W6_Plate.kicad_pcb (KiCad board)
At the start: 2 copper layers, 243.2 x 106 mm, 107 parts, among them J1 USB_C Main, J2 USB_C I2C_L, J3 USB_C I2C_R, SW1 SW_Push, SW10 SW_Push, SW11 SW_Push, SW12 SW_Push, SW13 SW_Push, SW14 SW_Push, SW15 SW_Push, SW16 SW_Push, SW17 SW_Push, SW18 SW_Push, SW19 SW_Push, SW2 SW_Push, SW20 SW_Push, SW21 SW_Push, SW22 SW_Push, SW23 SW_Push, SW24 SW_Push, SW25 SW_Push, SW26 SW_Push, SW27 SW_Push, SW28 SW_Push, SW29 SW_Push, SW3 SW_Push, SW30 SW_Push, SW31 SW_Push, SW32 SW_Push, SW33 SW_Push, SW34 SW_Push, SW35 SW_Push, SW36 SW_Push, SW37 SW_Push, SW4 SW_Push, SW5 SW_Push, SW6 SW_Push, SW7 SW_Push, SW8 SW_Push, SW9 SW_Push, U2 TCA9555RTWR, U3 ATmega32U4-MU, Y1 16MHZ

Commit message: Add: Plate PCB
Parts:
- removed C1, C2: 22nF, WetCorn:C_0402_HandSolder
- removed C3: 0.1u, WetCorn:C_0402_HandSolder
- removed C4, C5, C6, C7: 0.1uF, WetCorn:C_0402_HandSolder
- removed C8: 4.7uF, WetCorn:C_0402_HandSolder
- removed C9: 1uF, WetCorn:C_0402_HandSolder
- removed D1, D10, D11, D12, D13, D14, D15, D16, D17, D18, D19, D2, D20, D21, D22, D23, D24, D25, D26, D27, D28, D29, D3, D30, D31, D32, D33, D34, D35, D36, D37, D4, D5, D6, D7, D8, D9: D, WetCorn:D_SOD-323_HandSoldering
- removed F1: 500mA, Fuse:Fuse_1206_3216Metric_Pad1.42x1.75mm_HandSolder
- removed J1: USB_C Main, WetCorn:USB-C-12-Pin-MidMount
- removed J2: USB_C I2C_L, WetCorn:USB-C-12-Pin-MidMount
- removed J3: USB_C I2C_R, WetCorn:USB-C-12-Pin-MidMount
- removed R1, R2: 5.1k, WetCorn:R_0402_HandSolder
- removed R3, R4: 4.7k, WetCorn:R_0402_HandSolder
- removed R5, R8, R9: 10k, WetCorn:R_0402_HandSolder
- removed R6, R7: 22R, WetCorn:R_0402_HandSolder
- removed SW1: SW_Push, WetCorn:Micro_Push_Button_3x6x2.5mm
- removed SW10, SW11, SW12, SW13, SW14, SW15, SW16, SW17, SW18, SW19, SW2, SW20, SW21, SW22, SW23, SW24, SW25, SW26, SW27, SW28, SW29, SW3, SW30, SW31, SW32, SW34, SW35, SW36, SW4, SW5, SW6, SW7, SW8, SW9: SW_Push, WetCorn:Kailh_Choc_1u
- removed SW33, SW37: SW_Push, WetCorn:Kailh_Choc_1.5u
- removed U2: TCA9555RTWR, Package_DFN_QFN:WQFN-24-1EP_4x4mm_P0.5mm_EP2.45x2.45mm
- removed U3: ATmega32U4-MU, Package_DFN_QFN:QFN-44-1EP_7x7mm_P0.5mm_EP5.2x5.2mm
- removed Y1: 16MHZ, Oscillator:Oscillator_SMD_Abracon_ASE-4Pin_3.2x2.5mm
- added REF**: Plate_Hole, WetCorn:Plate_Hole, F.Cu at (222.5, 72.3)
- added REF**: Plate_Hole, WetCorn:Plate_Hole, F.Cu at (276.5, 64.3)
- added REF**: Plate_Hole, WetCorn:Plate_Hole, F.Cu at (276.5, 81.3)
- added REF**: Plate_Hole, WetCorn:Plate_Hole, F.Cu at (258.5, 38.3)
- added REF**: Plate_Hole, WetCorn:Plate_Hole, F.Cu at (240.5, 35.3)
- added REF**: Plate_Hole, WetCorn:Plate_Hole, F.Cu at (222.5, 38.3)
- added REF**: Plate_Hole, WetCorn:Plate_Hole, F.Cu at (204.5, 40.8)
- added REF**: Plate_Hole, WetCorn:Plate_Hole, F.Cu at (258.5, 55.3)
- added REF**: Plate_Hole, WetCorn:Plate_Hole, F.Cu at (240.5, 52.3)
- added REF**: Plate_Hole, WetCorn:Plate_Hole, F.Cu at (222.5, 55.3)
- added REF**: Plate_Hole, WetCorn:Plate_Hole, F.Cu at (258.5, 72.3)
- added REF**: Plate_Hole, WetCorn:Plate_Hole, F.Cu at (102.0, 94.2)
- added REF**: Plate_Hole, WetCorn:Plate_Hole, F.Cu at (204.5, 57.8)
- added REF**: Plate_Hole, WetCorn:Plate_Hole, F.Cu at (240.5, 69.3)
- added REF**: Plate_Hole, WetCorn:Plate_Hole, F.Cu at (123.3, 74.8)
- added REF**: Plate_Hole, WetCorn:Plate_Hole, F.Cu at (105.3, 55.3)
- added REF**: Plate_Hole, WetCorn:Plate_Hole, F.Cu at (105.3, 72.3)
- added REF**: Plate_Hole, WetCorn:Plate_Hole, F.Cu at (123.3, 57.8)
- added REF**: Plate_Hole, WetCorn:Plate_Hole, F.Cu at (87.3, 35.3)
- added REF**: Plate_Hole, WetCorn:Plate_Hole, F.Cu at (69.3, 55.3)
- added REF**: Plate_Hole, WetCorn:Plate_Hole, F.Cu at (123.3, 40.8)
- added REF**: Plate_Hole, WetCorn:Plate_Hole, F.Cu at (122.9, 96.4)
- added REF**: 3x6_PactSwitch_Hole, WetCorn:3x6_PactSwitch_Hole, F.Cu at (91.1, 94.8)
- added REF**: Plate_Hole, WetCorn:Plate_Hole, F.Cu at (69.3, 38.3)
- added REF**: Plate_Hole, WetCorn:Plate_Hole, F.Cu at (105.3, 38.3)
- added REF**: Plate_Hole, WetCorn:Plate_Hole, F.Cu at (204.5, 74.8)
- added REF**: Plate_Hole, WetCorn:Plate_Hole, F.Cu at (145.5, 101.1)
- added REF**: Plate_Hole, WetCorn:Plate_Hole, F.Cu at (87.3, 69.3)
- added REF**: Plate_Hole, WetCorn:Plate_Hole, F.Cu at (87.3, 52.3)
- added REF**: Plate_Hole, WetCorn:Plate_Hole, F.Cu at (51.3, 81.3)
- added REF**: Plate_Hole, WetCorn:Plate_Hole, F.Cu at (51.3, 47.3)
- added REF**: Plate_Hole, WetCorn:Plate_Hole, F.Cu at (69.3, 72.3)
- added REF**: Plate_Hole, WetCorn:Plate_Hole, F.Cu at (51.3, 64.3)
- added REF**: Plate_Hole, WetCorn:Plate_Hole, F.Cu at (182.3, 101.0)
- added REF**: Plate_Hole, WetCorn:Plate_Hole, F.Cu at (204.9, 96.3)
- added REF**: Plate_Hole, WetCorn:Plate_Hole, F.Cu at (225.8, 94.2)
- added REF**: Plate_Hole, WetCorn:Plate_Hole, F.Cu at (276.5, 47.3)
Routing:
- net +5V: track 175.0 -> 0.00 mm, vias 10 -> 0
- net /Row_R0: track 161.8 -> 0.00 mm, vias 2 -> 0
- net /Row_L0: track 154.6 -> 0.00 mm, vias 2 -> 0
- net /Row_R1: track 143.8 -> 0.00 mm, vias 2 -> 0
- net /Row_L1: track 137.8 -> 0.00 mm, vias 2 -> 0
- net /Row_R2: track 124.6 -> 0.00 mm
- net /Row_L2: track 119.2 -> 0.00 mm, vias 2 -> 0
- net /Col_L4: track 106.3 -> 0.00 mm
- net /Col_R4: track 99.5 -> 0.00 mm, vias 1 -> 0
- net /Col_L3: track 92.3 -> 0.00 mm
- net /Row_L3: track 87.7 -> 0.00 mm, vias 2 -> 0
- net /Col_R3: track 79.7 -> 0.00 mm, vias 1 -> 0
- net /Col_L2: track 78.1 -> 0.00 mm, vias 1 -> 0
- net /Col_L0: track 76.5 -> 0.00 mm
- net /Col_R0: track 74.5 -> 0.00 mm
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- removed copper zone on B.Cu, net GND
- removed copper zone on B.Cu, net VSS

Commit message: fixing some outlines
Parts:
- added G***: LOGO, WetCorn:Logo, F.Cu at (259.2, 85.9)
- added REF**: Logo_L, WetCorn:Logo_L, F.Cu at (73.3, 85.9)
Routing:
- added copper zone on F.Cu, net (none)
