File: pcb/3w6/3W6.kicad_pcb (KiCad board)
At the start: 2 copper layers, 243.2 x 106 mm, 113 parts, among them J1 USB_C Main, J2 USB_C I2C_L, J3 USB_C I2C_R, SW1 SW_Push, SW10 SW_Push, SW11 SW_Push, SW12 SW_Push, SW13 SW_Push, SW14 SW_Push, SW15 SW_Push, SW16 SW_Push, SW17 Trackball_Choc_Combi, SW18 SW_Push, SW19 SW_Push, SW2 SW_Push, SW20 SW_Push, SW21 SW_Push, SW22 SW_Push, SW23 SW_Push, SW24 SW_Push, SW25 SW_Push, SW26 SW_Push, SW27 SW_Push, SW28 SW_Push, SW29 SW_Push, SW3 SW_Push, SW30 SW_Push, SW31 SW_Push, SW32 SW_Push, SW33 SW_Push, SW34 SW_Push, SW35 SW_Push, SW36 SW_Push, SW37 SW_Push, SW4 SW_Push, SW5 SW_Push, SW6 SW_Push, SW7 SW_Push, SW8 SW_Push, SW9 SW_Push, U1 ATmega32U4-AU, U2 PCA9555PW, Y1 16MHZ

Commit message: increased version no to 2.1 to distinguish boards from different runs/changes
Other:
- board text added: "3W6 V2.1 20210728"
- board text removed: "3W6 V2.0 20210705"

Commit message: add combie footprint for atmega. Can be used with MU and AU variant
Parts:
- U1: footprint Package_QFP:TQFP-44_10x10mm_P0.8mm -> Weteor:AtMega32U4-Combie
- moved D2 0.09 mm to (276.5, 42.5)
- moved D3 0.09 mm to (276.5, 59.5)
- moved REF** 0.09 mm to (258.5, 29.1)
- moved C9 0.09 mm to (84.3, 76.9)
- moved D5 0.09 mm to (51.3, 42.5)
- moved U1 0.09 mm to (89.7, 83.6)
- moved Y1 0.09 mm to (78.8, 84.4)
- moved D18 0.09 mm to (87.3, 30.5)
- moved R1 0.09 mm to (55.4, 39.5)
- moved C3 0.09 mm to (237.7, 79.8)
- moved R9 0.09 mm to (99.0, 86.0)
- moved SW7 0.09 mm to (51.3, 81.2)
- moved D37 0.09 mm to (149.3, 103.8)
- moved REF** 0.09 mm to (105.2, 29.1)
- moved SW4 0.09 mm to (276.5, 81.2)
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Routing:
- net +5V: track 166.7 -> 193.8 mm, vias 6 -> 11
- net GND: track 30.4 -> 44.1 mm, vias 18 -> 29
- net /I2C_SDA_L: track 61.6 -> 67.3 mm
- net /I2C_SCL_L: track 59.5 -> 65.1 mm
- net /D-: track 63.2 -> 66.9 mm
- net /Col_L1: track 77.8 -> 81.3 mm
- net Net-(U1-Pad12): track 0.00 -> 3.45 mm
- net Net-(U1-Pad22): track 0.00 -> 3.23 mm
- net Net-(R9-Pad2): track 2.87 -> 6.06 mm
- net /Col_L0: track 75.7 -> 78.9 mm
- net /Row_L2: track 123.2 -> 126.2 mm
- net Net-(U1-Pad32): track 0.00 -> 3.07 mm
- net Net-(U1-Pad21): track 0.00 -> 3.07 mm
- net /Col_L2: track 77.6 -> 80.6 mm
- net /Row_L1: track 140.2 -> 143.1 mm
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- added copper zone on F.Cu, net GND
- added copper zone on F.Cu, net VSS
Other:
- outline, holes or cut-outs redrawn
- net class Default removed
- net class PWR removed
- board text added: "3W6 V2.2 20221017"
- board text removed: "3W6 V2.1 20210728"
